File: FC.kicad_pcb (KiCad board)
At the start: 6 copper layers, 50 x 50 mm, 117 parts, among them J1 USB4105-GF-A-120, J10 Conn_01x01, J11 Conn_01x01, J12 Conn_01x01, J13 Conn_01x01, J14 Conn_01x01, J15 Conn_01x01, J16 Conn_01x01, J17 Conn_01x01, J18 Conn_01x01, J19 Conn_01x01, J2 DM3AT-SF-PEJM5, J20 Conn_01x01, J21 Conn_01x01, J22 Conn_01x01, J23 Conn_01x01, J24 Conn_01x01, J25 Conn_01x01, J26 Conn_01x01, J27 Conn_01x01, J28 Conn_01x01, J3 CONMHF1-SMD-G-T, J30 Conn_01x01, J31 Conn_01x01, J32 Conn_01x01, J33 Conn_01x01, J34 Conn_01x08, J4 Conn_01x05, J5 Conn_01x01, J6 Conn_01x01, J7 Conn_01x01, J8 Conn_01x01, J9 Conn_01x01, U1 TLV76733DRVx, U10 STM32H757IITx, U11 ECS-TXO-2520-33-240-AN-TR, U12 4492, U13 4492, U14 4492, U15 4492, U16 4492, U17 PCM12SMTR, U19 LSM6DSOXTR, U2 AK09940A, U3 ICM-42688-P, U4 ICM-45686, U5 DPS368XTSA1, U6 TPS7A0218DBVR, U7 CDBURT0530LL-HF, U8 CDBURT0530LL-HF, U9 MAX-M10S

Commit message: V2 with feedback
Parts:
- removed U8: CDBURT0530LL-HF, Snapeda:CDBURT
- added R13: 100kR, Resistor_SMD:R_0603_1608Metric, F.Cu at (193.8, 59.5)
- added R5: 100kR, Resistor_SMD:R_0603_1608Metric, F.Cu at (191.2, 68.8)
- added U18: DMP2045U-7, Snapeda:SOT-23_DIO, F.Cu at (194.0, 68.5)
- added U21: USBLC6-2SC6, Package_TO_SOT_SMD:SOT-23-6, B.Cu at (189.5, 76.2)
- C1, C11, C12, C2, C26, C28, C29, C3, C39, C40, C42, C46, C47, C48, C49, C50, C51, C52, C53, C54, R10, R3, R4, R6, R8, R9, U6: moved to F.Cu
- U12, U13, U14, U15, U3, U4, U5: moved to B.Cu
- U7: value CDBURT0530LL-HF -> DMP2045U-7; footprint Snapeda:CDBURT -> Snapeda:SOT-23_DIO; moved to F.Cu
- moved U19 22.0 mm to (155.5, 81.0), turned to 180 degrees
- moved C49 20.5 mm to (155.2, 78.5)
- moved C47 20.0 mm to (152.5, 81.0), turned to 90 degrees
- moved U5 19.5 mm to (173.0, 64.0), turned to 0 degrees
- moved C41 19.0 mm to (194.0, 58.2), turned to 180 degrees
- moved C5 17.4 mm to (170.5, 64.2), turned to 90 degrees
- moved C4 16.5 mm to (173.0, 66.2)
- moved C6 15.0 mm to (167.0, 66.2), turned to 180 degrees
- moved C10 14.4 mm to (153.4, 68.6), turned to 0 degrees
- moved R9 13.2 mm to (189.5, 80.0)
- moved C7 12.6 mm to (167.8, 63.5)
- moved U3 11.8 mm to (156.2, 71.1), turned to 90 degrees
- moved C8 11.5 mm to (156.4, 68.6)
- moved C17 10.6 mm to (176.2, 64.8), turned to -90 degrees
- moved U4 10.3 mm to (165.5, 63.8), turned to -90 degrees
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Connections:
- C12 pad 1: Net-(U6-GND) -> GND
- C3 pad 1: Net-(U6-GND) -> GND
- C30 pad 1: +5V -> GND
- C30 pad 2: Net-(U1-EN) -> +5V
- J1 pad A4: Net-(J1-VBUS-PadA4) -> /USB_VBUS
- J1 pad A9: Net-(J1-VBUS-PadA4) -> /USB_VBUS
- R1 pad 2: Net-(J1-DN1) -> Net-(R1-Pad2)
- R2 pad 2: Net-(J1-DP1) -> Net-(R2-Pad2)
- U1 pad 4: Net-(U1-EN) -> +5V
- U1 pad 6: Net-(U1-EN) -> +5V
- U10 pad 156: IMU3_MISO -> BARO_MISO
- U10 pad 157: IMU3_SCL -> BARO_SCL
- U10 pad 158: IMU3_MOSI -> BARO_MOSI
- U10 pad 19: unconnected-(U10-PF1-Pad19) -> IMU1_INT
- U10 pad 2: IMU3_INT -> unconnected-(U10-PE3-Pad2)
- U10 pad 27: BARO_SCL -> IMU1_SCL
- U10 pad 28: BARO_MISO -> IMU1_MISO
- U10 pad 29: BARO_MOSI -> IMU1_MOSI
- U10 pad 34: IMU1_INT -> IMU3_INT
- U10 pad 35: IMU1_MOSI -> IMU3_MOSI
- U10 pad 36: IMU1_MISO -> IMU3_MISO
- U10 pad 78: IMU1_SCL -> IMU3_SCL
- U6 pad 2: Net-(U6-GND) -> GND
- U7 pad 1: +5V -> Net-(U7-G)
- U7 pad 2: Net-(J1-VBUS-PadA4) -> /ESC_5V
Routing:
- net GND: track 202.3 -> 169.3 mm, vias 72 -> 83
- net +3.3V: track 123.0 -> 147.8 mm, vias 48 -> 52
- net /USB_VBUS: track 0.00 -> 23.3 mm, vias 0 -> 1
- net IMU1_SCL: track 28.2 -> 6.61 mm, vias 2 -> 1
- net +5V: track 256.6 -> 236.0 mm, vias 11 -> 9
- net Net-(U15-DIN): track 6.69 -> 23.0 mm
- net /LEDC_PWM: track 17.0 -> 2.35 mm, vias 1 -> 0
- net Net-(J1-VBUS-PadA4): track 14.4 -> 0.00 mm, vias 2 -> 0
- net IMU3_SCL: track 14.9 -> 27.2 mm
- net IMU3_MISO: track 16.4 -> 5.88 mm
- net FSYNC: track 41.3 -> 32.0 mm
- net IMU2_SCL: track 12.7 -> 5.03 mm, vias 2 -> 1
- net IMU3_INT: track 12.0 -> 5.24 mm, vias 2 -> 0
- net IMU3_MOSI: track 13.8 -> 7.89 mm, vias 2 -> 0
- net Net-(U10-BOOT0): track 17.3 -> 11.7 mm, vias 1 -> 2
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- added copper zone on B.Cu, net GND
- added copper zone on In3.Cu, net GND
Other:
- board text removed: "*"

Commit message: V1 manufacturing
Parts:
- removed the C14 at (164.0, 61.2)
- removed the C36 at (167.0, 68.8)
- removed the C43 at (165.5, 68.8)
- removed the C44 at (166.2, 74.0)
- removed the C45 at (166.2, 72.5)
- removed L1: 2.2uH, Inductor_SMD:L_0603_1608Metric
- removed the R1 at (183.8, 75.2)
- removed the R2 at (183.8, 77.0)
- added C2: 100nF, Capacitor_SMD:C_0603_1608Metric, B.Cu at (163.0, 66.0)
- added C23: 100nF, Capacitor_SMD:C_0603_1608Metric, B.Cu at (161.2, 58.2)
- C31: value 2.2uF -> 4.7uF
- C47: renamed from C49; value 10nF -> 100nF
- moved R10 0.25 mm to (189.5, 80.2)
- moved C24 0.20 mm to (164.2, 58.2)
- turned J3 to 180 degrees
- renumbered C29 to C1, C23 to C10, C33 to C11, C22 to C12, C21 to C13, C20 to C14, C19 to C15, C39 to C16, C32 to C17, C34 to C19, C17 to C20, C16 to C21, C15 to C22, C35 to C24, C46 to C25, C13 to C26, C40 to C27, C41 to C28, C42 to C29, C28 to C3, C11 to C32, C54 to C33, C48 to C34, C53 to C35, C52 to C36, C51 to C37, C50 to C38, C3 to C39, C27 to C4, C12 to C40, C10 to C41, C8 to C42, C9 to C43, C6 to C44, C7 to C45, C47 to C46, C4 to C48, C5 to C49, C37 to C5, C2 to C50, C1 to C51, C38 to C6, C26 to C7, C25 to C8, C24 to C9, R7 to R1, R9 to R10, R6 to R11, R8 to R2, R4 to R3, R3 to R4, R13 to R5, R5 to R6, R11 to R7, R12 to R8, R10 to R9, U10 to U1, U18 to U10, U1 to U11, U6 to U12, U16 to U13, U15 to U14, U14 to U15, U12 to U16, U13 to U17, U17 to U18, U3 to U2, U4 to U3, U19 to U4, U9 to U6, U2 to U7, U11 to U8, U7 to U9
Connections:
- net Net-(U9-RF_IN) renamed /Sensors/RF_IN
- J1 pad S1: GND -> unconnected-(J1-GND-PadS1)_3
- U1 pad 15: Net-(U10-VLXSMPS) -> unconnected-(U1-VLXSMPS-Pad15)
- U1 pad 16: +3.3V -> GND
- U1 pad 17: Net-(U10-VFBSMPS) -> GND
- U1 pad 8: unconnected-(U10-VBAT-Pad8) -> +3.3V
- U21 pad 1: Net-(R2-Pad2) -> /USB_DP
- U21 pad 3: Net-(R1-Pad2) -> /USB_DN
Routing:
- net Net-(U10-VFBSMPS): track 9.46 -> 0.00 mm, vias 1 -> 0
- net Net-(U10-VLXSMPS): track 6.25 -> 0.00 mm, vias 1 -> 0
- net GND: track 169.3 -> 173.9 mm, vias 83 -> 108
- net +3.3V: track 147.8 -> 143.7 mm, vias 52 -> 51
- net Net-(R2-Pad2): track 4.02 -> 0.00 mm
- net Net-(R1-Pad2): track 3.81 -> 0.00 mm
- net /USB_DN: track 16.1 -> 14.0 mm
- net +5V: track 236.0 -> 237.5 mm
- net /Sensors/RF_IN: track 9.13 -> 8.24 mm
- net Net-(C29-Pad2): track 6.49 -> 7.12 mm
- net /USB_DP: track 19.3 -> 18.7 mm
- added copper zone on F.Cu, net GND
Other:
- board text added: "GigaFC H7"
- board text added: "JLCJLCJLCJLC"
- board text added: "v1 - 2425"
