File: FC.kicad_sch (KiCad schematic)
At the start: 98 parts, among them J1 USB4105-GF-A-120, J10 Conn_01x01, J11 Conn_01x01, J12 Conn_01x01, J13 Conn_01x01, J14 Conn_01x01, J15 Conn_01x01, J16 Conn_01x01, J17 Conn_01x01, J18 Conn_01x01, J19 Conn_01x01, J2 DM3AT-SF-PEJM5, J20 Conn_01x01, J21 Conn_01x01, J22 Conn_01x01, J23 Conn_01x01, J24 Conn_01x01, J25 Conn_01x01, J26 Conn_01x01, J27 Conn_01x01, J28 Conn_01x01, J30 Conn_01x01, J31 Conn_01x01, J32 Conn_01x01, J33 Conn_01x01, J34 Conn_01x08, J4 Conn_01x05, J5 Conn_01x01, J6 Conn_01x01, J7 Conn_01x01, J8 Conn_01x01, J9 Conn_01x01, U1 TLV76733DRVx, U10 STM32H757IITx, U11 ECS-TXO-2520-33-240-AN-TR, U12 4492, U13 4492, U14 4492, U15 4492, U16 4492, U17 PCM12SMTR, U6 TPS7A0218DBVR, U7 CDBURT0530LL-HF, U8 CDBURT0530LL-HF

Commit message: V2 with feedback
Parts:
- removed U7, U8: CDBURT0530LL-HF, Snapeda:CDBURT, symbol Snapeda:CDBURT0530LL-HF
- added R13, R5: 100kR, Resistor_SMD:R_0603_1608Metric, symbol Device:R_Small
- added U18, U7: DMP2045U-7, Snapeda:SOT-23_DIO, symbol Snapeda:DMP2045U-7
- added U21: USBLC6-2SC6, Package_TO_SOT_SMD:SOT-23-6, symbol Power_Protection:USBLC6-2SC6
Connections:
- net +5V: now also C30.2, U1.4 (EN), U1.6 (IN), U18.3 (D), U7.3 (D); no longer C30.1
- net BARO_MISO: now also U10.156 (PG12); no longer U10.28 (PF8)
- net BARO_MOSI: now also U10.158 (PG14); no longer U10.29 (PF9)
- net BARO_SCL: now also U10.157 (PG13); no longer U10.27 (PF7)
- net ESC_5V: now also U7.2 (S)
- net GND: now also C12.1, C3.1, C30.1, U6.2 (GND), R13.2, R5.2, U21.2 (GND)
- net IMU1_INT: now also U10.19 (PF1); no longer U10.34 (PC0)
- net IMU1_MISO: now also U10.28 (PF8); no longer U10.36 (PC2_C)
- net IMU1_MOSI: now also U10.29 (PF9); no longer U10.35 (PC1)
- net IMU1_SCL: now also U10.27 (PF7); no longer U10.78 (PB10)
- net IMU3_INT: now also U10.34 (PC0); no longer U10.2 (PE3)
- net IMU3_MISO: now also U10.36 (PC2_C); no longer U10.156 (PG12)
- net IMU3_MOSI: now also U10.35 (PC1); no longer U10.158 (PG14)
- net IMU3_SCL: now also U10.78 (PB10); no longer U10.157 (PG13)
- net USB_VBUS: now reaches J1.A4 (VBUS), J1.A9 (VBUS)
- net USB_VBUS: now also U18.2 (S), U21.5 (VBUS)
- net at J1.A6 (DP1), J1.B6 (DP2): now also U21.6 (I/O1); no longer R2.2
- net at J1.A7 (DN1), J1.B7 (DN2): now also U21.4 (I/O2); no longer R1.2
- new net: R13.1, U7.1 (G)
- new net: R2.2, U21.1 (I/O1)
- new net: R5.1, U18.1 (G)
- new net: R1.2, U21.3 (I/O2)
Other:
- note added: "3.3v"
- note added: "USB"
- note removed: "USB & 3.3V"
- title: (none) -> Flight Controller H7
- moved on the sheet: C30, C31, J1, R1, R11, R12, R2, U1

Commit message: V1 manufacturing
Parts:
- removed C36: 4.7uF, Capacitor_SMD:C_0603_1608Metric, symbol Device:C_Small
- removed C43: 220pF, Capacitor_SMD:C_0603_1608Metric, symbol Device:C_Small
- removed C44, C45: 10uF, Capacitor_SMD:C_0603_1608Metric, symbol Device:C_Small
- removed L1: 2.2uH, Inductor_SMD:L_0603_1608Metric, symbol Device:L_Small
- removed R1, R2: 22R, Resistor_SMD:R_0603_1608Metric, symbol Device:R_Small
- added C2: 100nF, Capacitor_SMD:C_0603_1608Metric, symbol Device:C_Small
- C31: value 2.2uF -> 4.7uF
- renumbered C29 to C1, C23 to C10, C33 to C11, C22 to C12, C21 to C13, C20 to C14, C19 to C15, C39 to C16, C32 to C17, C34 to C19, C17 to C20, C16 to C21, C15 to C22, C46 to C23, C35 to C24, C14 to C25, C13 to C26, C40 to C27, C41 to C28, C42 to C29, C28 to C3, C11 to C32, C54 to C33, C48 to C34, C53 to C35, C52 to C36, C51 to C37, C50 to C38, C3 to C39, C27 to C4, C12 to C40, C37 to C5, C38 to C6, C26 to C7, C25 to C8, C24 to C9, R7 to R1, R9 to R10, R8 to R2, R4 to R3, R3 to R4, R13 to R5, R5 to R6, R11 to R7, R12 to R8, R10 to R9, U10 to U1, U18 to U10, U1 to U11, U6 to U12, U16 to U13, U15 to U14, U14 to U15, U12 to U16, U13 to U17, U17 to U18, U11 to U8, U7 to U9
Connections:
- net +3.3V: now also U1.8 (VBAT), C2.2; no longer U1.16 (VDDSMPS)
- net GND: now also U1.16 (VDDSMPS), U1.17 (VFBSMPS), C2.1; no longer J1.S1 (GND)
- net USB_DN: now also U21.3 (I/O2)
- net USB_DP: now also U21.1 (I/O1)
- no-connect marks 11 -> 12
Other:
- moved on the sheet: C26, J12, R7, U18
