File: sensors.kicad_sch (KiCad schematic)
At the start: 19 parts, among them J3 CONMHF1-SMD-G-T, U19 LSM6DSOXTR, U2 AK09940A, U3 ICM-42688-P, U4 ICM-45686, U5 DPS368XTSA1, U9 MAX-M10S

Commit message: V1 manufacturing
Parts:
- C47: renamed from C49; value 10nF -> 100nF
- renumbered C10 to C41, C8 to C42, C9 to C43, C6 to C44, C7 to C45, C47 to C46, C4 to C48, C5 to C49, C2 to C50, C1 to C51, R6 to R11, U3 to U2, U4 to U3, U19 to U4, U9 to U6, U2 to U7
Connections:
- net RF_IN: now reaches J3.1, U6.11 (RF_IN)
Changed lines of the file:
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@@
 	(text "50R matched"
 		(exclude_from_sim no)
-		(at 267.208 49.276 0)
+		(at 275.082 47.498 0)
 		(effects
 			(font
@@
 		)
 	)
+	(label "RF_IN"
+		(at 264.16 50.8 0)
+		(effects
+			(font
+				(size 1.27 1.27)
+			)
+			(justify left bottom)
+		)
+	)
 	(global_label "MAG_MISO"
 		(shape input)
@@
 		(on_board yes)
 		(dnp no)
-		(property "Reference" "C10"
+		(property "Reference" "C41"
 			(at 21.59 35.56 90)
 			(effects
@@
 			(project "FC"
 				(path "/af6eb15d-b811-492c-ba2c-7b7824e394d5/40a622d2-e18b-4cb6-bade-298dc6c9c0f2"
-					(reference "C10")
+					(reference "C41")
 					(unit 1)
 				)
@@
 		(on_board yes)
 		(dnp no)
-		(property "Reference" "C47"
+		(property "Reference" "C46"
 			(at 115.57 115.57 90)
 			(effects
@@
 			(project "FC"
 				(path "/af6eb15d-b811-492c-ba2c-7b7824e394d5/40a622d2-e18b-4cb6-bade-298dc6c9c0f2"
-					(reference "C47")
+					(reference "C46")
 					(unit 1)
 				)
@@
 		(dnp no)
 		(fields_autoplaced yes)
-		(property "Reference" "U2"
-			(at 245.11 110.744 0)
+		(property "Reference" "U7"
+			(at 245.11 109.22 0)
 			(effects
 				(font
@@
 		)
 		(property "Value" "AK09940A"
-			(at 245.11 113.284 0)
+			(at 245.11 111.76 0)
 			(effects
 				(font
@@
 			(project "FC"
 				(path "/af6eb15d-b811-492c-ba2c-7b7824e394d5/40a622d2-e18b-4cb6-bade-298dc6c9c0f2"
-					(reference "U2")
+					(reference "U7")
 					(unit 1)
 				)
@@
 		(on_board yes)
 		(dnp no)
-		(property "Reference" "R6"
+		(property "Reference" "R11"
 			(at 220.726 55.88 90)
 			(effects
@@
 			(project "FC"
 				(path "/af6eb15d-b811-492c-ba2c-7b7824e394d5/40a622d2-e18b-4cb6-bade-298dc6c9c0f2"
-					(reference "R6")
+					(reference "R11")
 					(unit 1)
 				)
@@
 		(dnp no)
 		(fields_autoplaced yes)
-		(property "Reference" "U19"
-			(at 155.448 106.172 0)
+		(property "Reference" "U4"
+			(at 156.21 106.68 0)
 			(effects
 				(font
@@
 		)
 		(property "Value" "LSM6DSOXTR"
-			(at 155.448 108.712 0)
+			(at 156.21 109.22 0)
 			(effects
 				(font
@@
 			(project ""
 				(path "/af6eb15d-b811-492c-ba2c-7b7824e394d5/40a622d2-e18b-4cb6-bade-298dc6c9c0f2"
-					(reference "U19")
+					(reference "U4")
 					(unit 1)
 				)
@@
 		(on_board yes)
 		(dnp no)
-		(fields_autoplaced yes)
-		(property "Reference" "U9"
-			(at 247.2533 68.58 0)
+		(property "Reference" "U6"
+			(at 226.314 30.988 0)
 			(effects
 				(font
@@
 		)
 		(property "Value" "MAX-M10S"
-			(at 247.2533 71.12 0)
+			(at 223.266 33.528 0)
 			(effects
 				(font
@@
 			(project "FC"
 				(path "/af6eb15d-b811-492c-ba2c-7b7824e394d5/40a622d2-e18b-4cb6-bade-298dc6c9c0f2"
-					(reference "U9")
+					(reference "U6")
 					(unit 1)
 				)
@@
 		(on_board yes)
 		(dnp no)
-		(property "Reference" "C4"
+		(property "Reference" "C48"
 			(at 125.73 36.83 90)
 			(effects
@@
 			(project "FC"
 				(path "/af6eb15d-b811-492c-ba2c-7b7824e394d5/40a622d2-e18b-4cb6-bade-298dc6c9c0f2"
-					(reference "C4")
+					(reference "C48")
 					(unit 1)
 				)
@@
 		(on_board yes)
 		(dnp no)
-		(property "Reference" "C7"
+		(property "Reference" "C45"
 			(at 21.844 120.396 90)
 			(effects
@@
 			(project "FC"
 				(path "/af6eb15d-b811-492c-ba2c-7b7824e394d5/40a622d2-e18b-4cb6-bade-298dc6c9c0f2"
-					(reference "C7")
+					(reference "C45")
 					(unit 1)
 				)
@@
 		(on_board yes)
 		(dnp no)
-		(property "Reference" "C49"
+		(property "Reference" "C47"
 			(at 115.824 120.396 90)
 			(effects
@@
 			)
 		)
-		(property "Value" "10nF"
+		(property "Value" "100nF"
 			(at 121.158 120.396 90)
 			(effects
@@
 			(project "FC"
 				(path "/af6eb15d-b811-492c-ba2c-7b7824e394d5/40a622d2-e18b-4cb6-bade-298dc6c9c0f2"
-					(reference "C49")
+					(reference "C47")
 					(unit 1)
 				)
@@
 		(on_board yes)
 		(dnp no)
-		(property "Reference" "C9"
+		(property "Reference" "C43"
 			(at 21.844 44.196 90)
 			(effects
@@
 			(project "FC"
 				(path "/af6eb15d-b811-492c-ba2c-7b7824e394d5/40a622d2-e18b-4cb6-bade-298dc6c9c0f2"
-					(reference "C9")
+					(reference "C43")
 					(unit 1)
 				)
@@
 		(on_board yes)
 		(dnp no)
-		(property "Reference" "C8"
+		(property "Reference" "C42"
 			(at 21.59 39.37 90)
 			(effects
@@
 			(project "FC"
 				(path "/af6eb15d-b811-492c-ba2c-7b7824e394d5/40a622d2-e18b-4cb6-bade-298dc6c9c0f2"
-					(reference "C8")
+					(reference "C42")
 					(unit 1)
 				)
@@
 		(on_board yes)
 		(dnp no)
-		(property "Reference" "C5"
+		(property "Reference" "C49"
 			(at 125.984 41.656 90)
 			(effects
@@
 			(project "FC"
 				(path "/af6eb15d-b811-492c-ba2c-7b7824e394d5/40a622d2-e18b-4cb6-bade-298dc6c9c0f2"
-					(reference "C5")
+					(reference "C49")
 					(unit 1)
 				)
@@
 		(on_board yes)
 		(dnp no)
-		(property "Reference" "U4"
+		(property "Reference" "U3"
 			(at 62.738 106.68 0)
 			(effects
@@
 			(project "FC"
 				(path "/af6eb15d-b811-492c-ba2c-7b7824e394d5/40a622d2-e18b-4cb6-bade-298dc6c9c0f2"
-					(reference "U4")
+					(reference "U3")
 					(unit 1)
 				)
@@
 		(on_board yes)
 		(dnp no)
-		(property "Reference" "C6"
+		(property "Reference" "C44"
 			(at 21.59 115.57 90)
 			(effects
@@
 			(project "FC"
 				(path "/af6eb15d-b811-492c-ba2c-7b7824e394d5/40a622d2-e18b-4cb6-bade-298dc6c9c0f2"
-					(reference "C6")
+					(reference "C44")
 					(unit 1)
 				)
@@
 		(on_board yes)
 		(dnp no)
-		(property "Reference" "C2"
+		(property "Reference" "C50"
 			(at 213.614 117.856 90)
 			(effects
@@
 			(project "FC"
 				(path "/af6eb15d-b811-492c-ba2c-7b7824e394d5/40a622d2-e18b-4cb6-bade-298dc6c9c0f2"
-					(reference "C2")
+					(reference "C50")
 					(unit 1)
 				)
@@
 		(on_board yes)
 		(dnp no)
-		(property "Reference" "C1"
+		(property "Reference" "C51"
 			(at 213.614 133.096 90)
 			(effects
@@
 			(project "FC"
 				(path "/af6eb15d-b811-492c-ba2c-7b7824e394d5/40a622d2-e18b-4cb6-bade-298dc6c9c0f2"
-					(reference "C1")
+					(reference "C51")
 					(unit 1)
 				)
@@
 		(on_board yes)
 		(dnp no)
-		(property "Reference" "U3"
+		(property "Reference" "U2"
 			(at 64.262 31.242 0)
 			(effects
@@
 			(project "FC"
 				(path "/af6eb15d-b811-492c-ba2c-7b7824e394d5/40a622d2-e18b-4cb6-bade-298dc6c9c0f2"
-					(reference "U3")
+					(reference "U2")
 					(unit 1)
 				)
